File: schematic.kicad_pcb (KiCad board)
At the start: 2 copper layers, 69.6 x 93.2 mm, 18 parts, among them J1 Conn_01x02_Socket, U1 NE555P, U2 4017

Commit message: Add files via upload
Parts:
- moved D11 52.2 mm to (27.5, 37.5)
- moved D7 52.0 mm to (42.0, 70.0)
- moved D3 48.2 mm to (68.0, 42.0)
- moved D4 30.4 mm to (62.0, 66.0)
- moved D1 27.0 mm to (56.5, 36.5)
- moved D2 19.7 mm to (63.0, 37.0)
- moved D9 19.7 mm to (36.0, 73.5)
- moved D5 19.1 mm to (68.5, 66.0)
- moved RV1 16.8 mm to (37.5, 40.1)
- moved C2 12.2 mm to (47.0, 60.5)
- moved R2 10.1 mm to (36.2, 59.0)
- moved J1 10.1 mm to (56.5, 63.0)
- moved D10 9.24 mm to (32.5, 66.5)
- moved U1 7.21 mm to (57.2, 46.7)
- moved D6 5.96 mm to (65.0, 73.5)
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Routing:
- net Net-(D4-A): track 29.0 -> 171.2 mm
- net Net-(D5-A): track 46.3 -> 163.5 mm
- net Net-(D6-A): track 41.8 -> 128.6 mm
- net Net-(D7-A): track 30.1 -> 88.3 mm
- net GND: track 75.9 -> 123.1 mm
- net Net-(D1-K): track 171.7 -> 132.5 mm
- net Net-(U1-DISCH): track 66.1 -> 43.4 mm
- net Net-(U1-CONT): track 43.4 -> 21.5 mm
- net Net-(D9-A): track 25.2 -> 46.0 mm
- net Net-(D10-A): track 27.4 -> 43.0 mm
- net Net-(D1-A): track 30.6 -> 18.7 mm
- net TR: track 53.8 -> 63.8 mm
- net Net-(D11-A): track 29.2 -> 34.5 mm
- net +5V: track 45.7 -> 50.5 mm
- net OUT: track 8.37 -> 5.36 mm
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